File: Arduino_Pro_Mini_XL.kicad_pcb (KiCad board)
At the start: 2 copper layers, 18.5 x 33.3 mm, 21 parts, among them M1 ARDUINO-PRO-MINI-XL, SW1 Reset, U1 ATmega1284P-MU, Y1 20MHz

Commit message: project files updated to Kicad version 9.0.1
Other:
- board text added: "by MPro: v${REVISION}"
- board text removed: "by MPro: v1.1"
